File: si-hardware-ais-mdm/power_input.kicad_sch (KiCad schematic)
At the start: 17 parts, among them Q1 IRLML6401, U1 LMR14206

Commit message: schematic  to pcb
Connections:
- net V_USB is gone; now on net VD: Q1.1 (G)
- net +3.3V: now also C6.1, C7.1, C8.1, L1.1, R3.1
- net at C2.1: now also C1.1, C3.1, C4.1, D1.2 (K), Q1.2 (S), R2.2, U1.5 (VIN)
- net GND: now reaches C2.2
- net GND: now also C1.2, C3.2, C4.2, C6.2, C7.2, C8.2, D2.2 (A), R1.2, R4.2, U1.2 (GND)
- net at R3.2: now also R4.1, U1.3 (FB)
- net at R2.1: now also U1.4 (~{SHDN})
- net at D2.1 (K): now also C5.2, U1.6 (SW)
- net at U1.1 (CB): now also C5.1, L1.2
- net VD: now reaches D1.1 (A)
- net VD: now also R1.1
