File: si-hardware-ais-mdm/MCU.kicad_sch (KiCad schematic)
At the start: 27 parts, among them J4 USB_C_Receptacle_USB2.0_16P, SW1 SW_Push, SW2 SW_Push, U6 ESP32-C6-MINI-1-H4, U7 LIS331HH, U9 24AA02E-OT

Commit message: routing final
Parts:
- added J5: Conn_01x03_Socket, Connector_PinHeader_2.54mm:PinHeader_1x03_P2.54mm_Horizontal, symbol Connector:Conn_01x03_Socket
Connections:
- net GND: now also J5.3 (Pin_3)
- net RX0 renamed mdm.SDN1
- net mdm.SDN1: now also J5.2 (Pin_2)
- net TX0 renamed mdm.SDN2
- net mdm.SDN2: now also J5.1 (Pin_1)
Changed lines of the file:
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@@
 	(wire
 		(pts
+			(xy 168.91 71.12) (xy 204.47 71.12)
+		)
+		(stroke
+			(width 0)
+			(type default)
+		)
+	)
+	(wire
+		(pts
 			(xy 125.73 93.98) (xy 138.43 93.98)
 		)
@@
 	(wire
 		(pts
+			(xy 179.07 114.3) (xy 193.04 114.3)
+		)
+		(stroke
+			(width 0)
+			(type default)
+		)
+	)
+	(wire
+		(pts
 			(xy 62.23 80.01) (xy 71.12 80.01)
 		)
@@
 	(wire
 		(pts
+			(xy 193.04 123.19) (xy 193.04 119.38)
+		)
+		(stroke
+			(width 0)
+			(type default)
+		)
+	)
+	(wire
+		(pts
 			(xy 262.89 105.41) (xy 255.27 105.41)
 		)
@@
 	(wire
 		(pts
-			(xy 168.91 71.12) (xy 204.47 71.12)
-		)
-		(stroke
-			(width 0)
-			(type default)
-		)
-	)
-	(wire
-		(pts
 			(xy 228.6 67.31) (xy 232.41 67.31)
 		)
@@
 	(wire
 		(pts
-			(xy 168.91 68.58) (xy 204.47 68.58)
-		)
-		(stroke
-			(width 0)
-			(type default)
-		)
-	)
-	(wire
-		(pts
 			(xy 92.71 109.22) (xy 92.71 99.06)
 		)
@@
 	(wire
 		(pts
+			(xy 179.07 116.84) (xy 193.04 116.84)
+		)
+		(stroke
+			(width 0)
+			(type default)
+		)
+	)
+	(wire
+		(pts
 			(xy 125.73 162.56) (xy 140.97 162.56)
 		)
@@
 	(wire
 		(pts
+			(xy 168.91 68.58) (xy 204.47 68.58)
+		)
+		(stroke
+			(width 0)
+			(type default)
+		)
+	)
+	(wire
+		(pts
 			(xy 186.69 78.74) (xy 189.23 78.74)
 		)
@@
 		)
 	)
+	(label "mdm.SDN2"
+		(at 179.07 114.3 0)
+		(fields_autoplaced yes)
+		(effects
+			(font
+				(size 1.27 1.27)
+			)
+			(justify left bottom)
+		)
+	)
 	(label "mdm.NSS2"
 		(at 125.73 81.28 0)
@@
 	)
 	(label "mdm.SDN2"
-		(at 168.91 68.58 270)
+		(at 171.45 68.58 0)
 		(fields_autoplaced yes)
 		(effects
@@
 				(size 1.27 1.27)
 			)
-			(justify right bottom)
+			(justify left bottom)
 		)
 	)
@@
 	)
 	(label "mdm.SDN1"
-		(at 168.91 71.12 0)
+		(at 171.45 71.12 0)
 		(fields_autoplaced yes)
 		(effects
@@
 		)
 	)
-	(label "mdm.GP2"
-		(at 125.73 78.74 0)
+	(label "mdm.SDN1"
+		(at 179.07 116.84 0)
 		(fields_autoplaced yes)
 		(effects
@@
 		)
 	)
-	(label "mdm.MISO"
-		(at 168.91 99.06 0)
+	(label "mdm.GP2"
+		(at 125.73 78.74 0)
 		(fields_autoplaced yes)
 		(effects
@@
 		)
 	)
-	(global_label "SDA"
-		(shape input)
-		(at 180.34 88.9 0)
+	(label "mdm.MISO"
+		(at 168.91 99.06 0)
 		(fields_autoplaced yes)
 		(effects
@@
 				(size 1.27 1.27)
 			)
-			(justify left)
-		)
-		(property "Intersheetrefs" "${INTERSHEET_REFS}"
-			(at 186.8933 88.9 0)
-			(effects
-				(font
-					(size 1.27 1.27)
-				)
-				(justify left)
-				(hide yes)
-			)
+			(justify left bottom)
 		)
 	)
-	(global_label "RX0"
+	(global_label "SDA"
 		(shape input)
-		(at 193.04 71.12 90)
+		(at 180.34 88.9 0)
 		(fields_autoplaced yes)
 		(effects
@@
 		)
 		(property "Intersheetrefs" "${INTERSHEET_REFS}"
-			(at 193.04 64.4458 90)
+			(at 186.8933 88.9 0)
 			(effects
 				(font
@@
 		)
 	)
-	(global_label "EN"
-		(shape input)
-		(at 213.36 118.11 0)
-		(fields_autoplaced yes)
-		(effects
-			(font
-				(size 1.27 1.27)
-			)
-			(justify left)
-		)
-		(property "Intersheetrefs" "${INTERSHEET_REFS}"
-			(at 218.8247 118.11 0)
-			(effects
-				(font
-					(size 1.27 1.27)
-				)
-				(justify left)
-				(hide yes)
-			)
-		)
-	)
-	(global_label "TX0"
-		(shape input)
-		(at 213.36 113.03 0)
-		(fields_autoplaced yes)
-		(effects
-			(font
-				(size 1.27 1.27)
-			)
-			(justify left)
-		)
-		(property "Intersheetrefs" "${INTERSHEET_REFS}"
-			(at 219.7318 113.03 0)
-			(effects
-				(font
-					(size 1.27 1.27)
-				)
-				(justify left)
-				(hide yes)
-			)
-		)
-	)
-	(global_label "TX0"
-		(shape input)
-		(at 187.96 68.58 90)
-		(fields_autoplaced yes)
-		(effects
-			(font
-				(size 1.27 1.27)
-			)
-			(justify left)
-		)
-		(property "Intersheetrefs" "${INTERSHEET_REFS}"
-			(at 187.96 62.2082 90)
-			(effects
-				(font
-					(size 1.27 1.27)
-				)
-				(justify left)
-				(hide yes)
-			)
-		)
-	)
 	(global_label "SCL"
 		(shape input)
@@
 		)
 	)
-	(global_label "RX0"
-		(shape input)
-		(at 213.36 115.57 0)
-		(fields_autoplaced yes)
-		(effects
-			(font
-				(size 1.27 1.27)
-			)
-			(justify left)
-		)
-		(property "Intersheetrefs" "${INTERSHEET_REFS}"
-			(at 220.0342 115.57 0)
-			(effects
-				(font
-					(size 1.27 1.27)
-				)
-				(justify left)
-				(hide yes)
-			)
-		)
-	)
 	(hierarchical_label "mdm_ais"
 		(shape input)
@@
 	(symbol
 		(lib_id "power:GNDD")
-		(at 213.36 120.65 90)
+		(at 193.04 123.19 0)
 		(unit 1)
 		(exclude_from_sim no)
@@
 		(fields_autoplaced yes)
 		(property "Reference" "#PWR067"
-			(at 219.71 120.65 0)
+			(at 193.04 129.54 0)
 			(effects
 				(font
@@
 		)
 		(property "Value" "GNDD"
-			(at 217.17 120.6499 90)
+			(at 195.58 124.2694 0)
 			(effects
 				(font
 					(size 1.27 1.27)
 				)
-				(justify right)
+				(justify left)
 			)
 		)
 		(property "Footprint" ""
-			(at 213.36 120.65 0)
+			(at 193.04 123.19 0)
 			(effects
 				(font
@@
 		)
 		(property "Datasheet" ""
-			(at 213.36 120.65 0)
+			(at 193.04 123.19 0)
 			(effects
 				(font
@@
 		)
 		(property "Description" "Power symbol creates a global label with name \"GNDD\" , digital ground"
-			(at 213.36 120.65 0)
+			(at 193.04 123.19 0)
 			(effects
 				(font
@@
 	)
 	(symbol
+		(lib_id "Connector:Conn_01x03_Socket")
+		(at 198.12 116.84 0)
+		(unit 1)
+		(exclude_from_sim no)
+		(in_bom yes)
+		(on_board yes)
+		(dnp no)
+		(fields_autoplaced yes)
+		(property "Reference" "J5"
+			(at 199.39 115.5699 0)
+			(effects
+				(font
+					(size 1.27 1.27)
+				)
+				(justify left)
+			)
+		)
+		(property "Value" "Conn_01x03_Socket"
+			(at 199.39 118.1099 0)
+			(effects
+				(font
+					(size 1.27 1.27)
+				)
+				(justify left)
+			)
+		)
+		(property "Footprint" "Connector_PinHeader_2.54mm:PinHeader_1x03_P2.54mm_Horizontal"
+			(at 198.12 116.84 0)
+			(effects
+				(font
+					(size 1.27 1.27)
+				)
+				(hide yes)
+			)
+		)
+		(property "Datasheet" "~"
+			(at 198.12 116.84 0)
+			(effects
+				(font
+					(size 1.27 1.27)
+				)
+				(hide yes)
+			)
+		)
+		(property "Description" "Generic connector, single row, 01x03, script generated"
+			(at 198.12 116.84 0)
+			(effects
+				(font
+					(size 1.27 1.27)
+				)
+				(hide yes)
+			)
+		)
+		(pin "2"
+		)
+		(pin "3"
+		)
+		(pin "1"
+		)
+		(instances
+			(project ""
+				(path "/97f80214-d5cc-4a35-9cac-bb1ff8330c6a/487f8325-78ac-466b-85b4-df92bc0f13d9"
+					(reference "J5")
+					(unit 1)
+				)
+			)
+		)
+	)
+	(symbol
 		(lib_id "Device:C")
 		(at 111.76 64.77 180)
@@
 					(unit 1)
 				)
-			)
-		)
-	)
-	(symbol
-		(lib_id "power:+3.3V")
-		(at 213.36 123.19 270)
-		(unit 1)
-		(exclude_from_sim no)
-		(in_bom yes)
-		(on_board yes)
-		(dnp no)
-		(fields_autoplaced yes)
-		(property "Reference" "#PWR064"
-			(at 209.55 123.19 0)
-			(effects
-				(font
-					(size 1.27 1.27)
-				)
-				(hide yes)
-			)
-		)
-		(property "Value" "+3.3V"
-			(at 217.17 123.1899 90)
-			(effects
-				(font
-					(size 1.27 1.27)
-				)
-				(justify left)
-			)
-		)
-		(property "Footprint" ""
-			(at 213.36 123.19 0)
-			(effects
-				(font
-					(size 1.27 1.27)
-				)
-				(hide yes)
-			)
-		)
-		(property "Datasheet" ""
-			(at 213.36 123.19 0)
-			(effects
-				(font
-					(size 1.27 1.27)
-				)
-				(hide yes)
-			)
-		)
-		(property "Description" "Power symbol creates a global label with name \"+3.3V\""
-			(at 213.36 123.19 0)
-			(effects
-				(font
-					(size 1.27 1.27)
-				)
-				(hide yes)
-			)
-		)
-		(pin "1"
-		)
-		(instances
-			(project "si-hardware-ais-mdm"
-				(path "/97f80214-d5cc-4a35-9cac-bb1ff8330c6a/487f8325-78ac-466b-85b4-df92bc0f13d9"
-					(reference "#PWR064")
-					(unit 1)
-				)

Commit message: added schematic pdf
Parts:
- removed R14, R23: 4.7K, Resistor_SMD:R_0402_1005Metric, symbol Device:R
- removed R21: 5K1, Resistor_SMD:R_0402_1005Metric, symbol Device:R
- removed U7: LIS331HH, Package_LGA:LGA-16_3x3mm_P0.5mm_LayoutBorder3x5y, symbol Sensor_Motion:LIS331HH
- removed U9: 24AA02E-OT, Package_TO_SOT_SMD:SOT-23-5, symbol Memory_EEPROM:24AA02E-OT
- added C40: 104/10V, Capacitor_SMD:C_0603_1608Metric, symbol Device:C
- added C41: 10uF/10V, Capacitor_SMD:C_0603_1608Metric, symbol Device:C
- added U9: STM32L432KBUx, Package_DFN_QFN:QFN-32-1EP_5x5mm_P0.5mm_EP3.45x3.45mm, symbol MCU_ST_STM32L4:STM32L432KBUx
- added Y3: 32.768KHz, Crystal:Crystal_SMD_3215-2Pin_3.2x1.5mm, symbol Device:Crystal
- C37, C38: value 10uF/10V -> 10pF; footprint Capacitor_SMD:C_0603_1608Metric -> Capacitor_SMD:C_0402_1005Metric
- C39: value 104/10V -> 1uF/10V; footprint Capacitor_SMD:C_0402_1005Metric -> Capacitor_SMD:C_0603_1608Metric
- R22: value 5K1 -> 10K
Connections:
- net +3.3V: now also C39.2, R22.2, C40.2, C41.2, U9.1 (VDD), U9.17 (VDD), U9.5 (VDDA); no longer C37.2, C38.2, C39.1, R22.1
- net D+: now also R18.2; no longer R17.2
- net D-: now also R17.2; no longer R18.2
- net GND: now also C37.2, C38.2, C39.1, C40.1, C41.1, U9.16 (VSS), U9.32 (VSS), U9.33 (VSS); no longer C37.1, C38.1, C39.2
- net i+: now also R18.1, U9.22 (PA12); no longer R17.1, U6.18 (IO13)
- net i-: now also R17.1, U9.21 (PA11); no longer R18.1, U6.17 (IO12)
- net mdm.CTS2: now also U9.10 (PA4); no longer U6.12 (IO0)
- net mdm.GP1: now also U9.28 (PB5); no longer U6.22 (IO8)
- net mdm.GP2: now also U9.29 (PB6); no longer U6.13 (IO1)
- net mdm.IRQ2: now also U9.30 (PB7); no longer U6.6 (IO3)
- net mdm.MISO: now also U9.12 (PA6); no longer U6.29 (IO23)
- net mdm.MOSI: now also U9.13 (PA7); no longer U6.28 (IO22)
- net mdm.NSS1: now also U9.25 (PA15); no longer U6.19 (IO14)
- net mdm.NSS2: no longer U6.5 (IO2)
- net mdm.RXCLK1: now also U9.15 (PB1); no longer U6.16 (IO7)
- net mdm.RXCLK2: now also U9.26 (PB3); no longer U6.10 (IO5)
- net mdm.RXDATA1: now also U9.14 (PB0); no longer U6.15 (IO6)
- net mdm.RXDATA2: now also U9.27 (PB4); no longer U6.9 (IO4)
- net mdm.SCLK: now also U9.11 (PA5); no longer U6.27 (IO21)
- net mdm.SDN1: now also U9.18 (PA8); no longer J5.2 (Pin_2), TP2.1, U6.30 (RXD0)
- net mdm.SDN2: now also U9.6 (PA0); no longer J5.1 (Pin_1), TP1.1, U6.31 (TXD0)
- net mdm.CTS1: no longer names the net of U6.26 (IO20)
- net mdm.IRQ1: no longer names the net of U6.20 (IO15)
- new net: TP1.1, U6.31 (TXD0)
- new net: C37.1, U9.2 (PC14), Y3.2
- new net: TP2.1, U6.30 (RXD0)
- new net: R22.1, U9.4 (NRST)
- new net: C38.1, U9.3 (PC15), Y3.1
- new net BOOT0: U9.31 (PH3)
- new net SWC: U9.24 (PA14)
- new net SWD: U9.23 (PA13)
- new net UART1_RX: U9.20 (PA10)
- new net UART1_TX: U9.19 (PA9)
- new net UART2_RX: U9.9 (PA3)
- new net UART2_TX: U9.8 (PA2)
- no-connect marks 2 -> 0
Other:
- moved on the sheet: C33, SW2
