File: si-hardware-ais-mdm/MCU.kicad_sch (KiCad schematic)
At the start: 27 parts, among them J4 USB_C_Receptacle_USB2.0_16P, J5 Conn_01x03_Socket, SW1 SW_Push, SW2 SW_Push, U6 ESP32-C6-MINI-1-H4, U9 STM32L432KBUx, Y3 32.768KHz

Commit message: change mcu control
Parts:
- removed J5: Conn_01x03_Socket, Connector_PinHeader_2.54mm:PinHeader_1x03_P2.54mm_Horizontal, symbol Connector:Conn_01x03_Socket
- removed R22: 10K, Resistor_SMD:R_0402_1005Metric, symbol Device:R
- removed TP1, TP2: TestPoint, TestPoint:TestPoint_Pad_D1.0mm, symbol Connector:TestPoint
- removed U9: STM32L432KBUx, Package_DFN_QFN:QFN-32-1EP_5x5mm_P0.5mm_EP3.45x3.45mm, symbol MCU_ST_STM32L4:STM32L432KBUx
- added 1M: 1M, Resistor_SMD:R_0402_1005Metric, symbol Device:R
- added C43: 22pF, Capacitor_SMD:C_0402_1005Metric, symbol Device:C
- added C44: 104/10V, Capacitor_SMD:C_0402_1005Metric, symbol Device:C
- added C45: 10uF/10V, CTS_Capacitor_SMD:C_0402_1005Metric, symbol Device:C
- added C46, C47: 104/10V, CTS_Capacitor_SMD:C_0402_1005Metric, symbol Device:C
- added D6, D7: 1N4148W, Diode_SMD:D_SOD-123, symbol Diode:1N4148W
- added J5: Conn_01x03_Pin, symbol Connector:Conn_01x03_Pin
- added R23, R27: 10K, Resistor_SMD:R_0402_1005Metric, symbol Device:R
- added U9: ~, symbol SI_MCU:STM32l496VET6
- added Y4: 8MHz, Crystal:Crystal_SMD_5032-2Pin_5.0x3.2mm, symbol Device:Crystal
- C32, C34, C35, C36, C39, C40, C41: footprint Capacitor_SMD:C_0603_1608Metric -> CTS_Capacitor_SMD:C_0402_1005Metric
- C33: value 104/10V -> 22pF
Connections:
- net +3.3V: now also R23.2, R27.1, U9.100 (VDD), U9.11 (VDD), U9.28 (VDD), U9.50 (VDD), U9.75 (VDD)
- net BOOT0: now also U9.94 (PH3)
- net GND: now also C43.2, C44.2, C45.1, C46.1, C47.1, J5.3 (Pin_3), U9.10 (VSS), U9.19 (VSSA), U9.27 (VSS), U9.49 (VSS), U9.74 (VSS), U9.99 (VSS)
- net SWC: now also J5.1 (Pin_1), U9.76 (PA14)
- net SWD: now also J5.2 (Pin_2), U9.72 (PA13)
- net i+: now also U9.71 (PA12(DP))
- net i-: now also U9.70 (PA11(DM))
- net mdm.CTS2: now also U9.57 (PD10)
- net mdm.GP1: now also U9.4 (PE5)
- net mdm.GP2: now also U9.5 (PE6)
- net mdm.IRQ2: now also U9.55 (PD8)
- net mdm.MISO: now also U9.31 (PA6(MISO))
- net mdm.MOSI: now also U9.32 (PA7(MOSI/I2C3_SCL))
- net mdm.NSS1: now also U9.37 (PB2)
- net mdm.RXCLK1: now also U9.36 (PB1)
- net mdm.RXCLK2: now also U9.17 (PC2(MISO))
- net mdm.RXDATA1: now also U9.35 (PB0)
- net mdm.RXDATA2: now also U9.18 (PC3)
- net mdm.SCLK: now also U9.24 (PA1(SCK/RX4))
- net mdm.SDN1: now also U9.90 (PB4)
- net mdm.SDN2: now also U9.89 (PB3)
- net DEBUG_ESP_TX: now reaches U6.31 (TXD0)
- net OSC32_IN: now reaches C37.1, Y3.2
- net OSC32_IN: now also U9.8 (PC14(OSC32_IN))
- net DEBUG_ESP_RX: now reaches U6.30 (RXD0)
- net OSC32_OUT: now reaches C38.1, Y3.1
- net OSC32_OUT: now also U9.9 (PC15(OSC32_OUT))
- net ESP_TX: now reaches U6.28 (IO22)
- net ESP_TX: now also U9.26 (PA3(UART2_RX))
- net ESP_RX: now reaches U6.29 (IO23)
- net ESP_RX: now also U9.25 (PA2(UART2_TX))
- net SCL: no longer names the net of U6.24 (IO18)
- net SDA: no longer names the net of U6.25 (IO19)
- new net: C45.2, C46.2, R27.2, U9.22 (VDDA), U9.73 (VDDUSB)
- new net OSC_IN: 1M.2, C33.1, U9.12 (PH0(OSC_IN)), Y4.2
- new net OSC_OUT: 1M.1, C43.1, U9.13 (PH1(OSC_OUT)), Y4.1
- new net RESET: C44.1, R23.1, SW2.2, U9.14 (NRST)
- new net VBAT: C47.2, D6.1 (K), D7.1 (K), U9.6 (VBAT)
- new net VBAT+: D6.2 (A), D7.2 (A)
- new net mdm.CTS1: U9.3 (PE4)
- new net mdm.IRQ1: U9.87 (PD6)
- new net peri.GPS_PPS: U9.56 (PD9)
- new net peri.GPS_RST: U9.81 (PD0)
- new net peri.GPS_RX: U9.68 (PA9(UART1_TX))
- new net peri.GPS_TX: U9.69 (PA10(UART1_RX))
- new net peri.SCL: U9.92 (PB6(I2C1_SCL))
- new net peri.SDA: U9.93 (PB7(I2C1_SDA))
- now unconnected: U6.23 (IO9)
Other:
- moved on the sheet: C31, C32, C34, C35, C36, C37, C38, C39, C40, C41, J4, R15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
